File: hardware/variant-b/env-sensor-b.kicad_pcb (KiCad board)
At the start: 4 copper layers, 28 x 51 mm, 58 parts, among them J1 USB-C 16P, J2 JST-PH 2P, SW1 SW_PROV, U1 ESP32-C6-MINI-1-N4, U2 SHT45-AD1F, U3 TPS62840DLC, U4 BQ24074RGTR, U5 USBLC6-2SC6

Commit message: build: add make pipeline, DRC gate and manufacturing outputs
KiCad 10 is available now, so the generated boards get checked and exported by
KiCad itself rather than only by the generator's own rules.

kicad-cli found what the offline checks could not, and the generator is fixed at
source in every case:
- a nested (justify) token stopped the boards loading at all
- the RF keep-out was drawn 2 mm into the module body, so it swallowed the
  module's own ground pads; it now spans the full board width and stops exactly
  at the antenna boundary, which is also the correct RF answer
- the USB-C receptacle's through-hole shield lugs were shorting a bottom-side
  pogo pad: the offline checker had assumed bottom pads can never collide with
  top parts, which is false for THT
- island trace edge clearance ignored half the trace width
- plane vias landed inside the sensor quiet zone and clashed with a later route
- the GND pour reached the module's 20 ground pads through single thermal
  spokes; GND now connects solid
- reference designators came off the silkscreen (F.Fab already carries them all)

231 violations -> 5 and 4, zero errors on both variants. Adds a GND stitching
ring, a Makefile as the single build entry point, a DRC gate with a written
policy for the three accepted warnings and a ratsnest budget that may only
decrease, a BOM/netlist generator from the shared model, and full fab outputs:
4-layer gerbers, Excellon drill, CPL, assembly PDF and STEP.
Parts:
- moved C11 26.9 mm to (119.9, 90.2)
- moved R1 18.6 mm to (106.0, 66.5), turned to 0 degrees
- moved C4 17.9 mm to (122.0, 66.5), turned to 0 degrees
- moved C3 15.3 mm to (121.5, 76.8)
- moved C1 14.2 mm to (106.0, 76.0), turned to 90 degrees
- moved C13 12.6 mm to (122.3, 90.2)
- moved C14 12.0 mm to (103.5, 90.5)
- moved C5 9.57 mm to (117.0, 91.2)
- moved C9 9.00 mm to (124.2, 75.0)
- moved R2 7.40 mm to (104.8, 78.5)
- moved TP14 7.13 mm to (111.5, 84.6)
- moved TP16 7.13 mm to (116.6, 84.6)
- moved TP2 7.13 mm to (111.5, 79.5)
- moved TP4 7.13 mm to (116.6, 79.5)
- moved TP1 7.13 mm to (109.0, 79.5)
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Routing:
- net GND: track 23.2 -> 31.3 mm, vias 1 -> 12
- net +3V0: track 20.7 -> 24.3 mm
Other:
- board text added: "ENV"
- board text added: "SENSOR"
- board text added: "VARIANT B"
- board text removed: "BAT"
- board text removed: "ENV SENSOR"
- board text removed: "VAR THERMALLY ISOLATED"
